File: GoProControl/goprocontrol.sch (EAGLE design)
At the start: 19 parts

Commit message: small board tweaks
Parts:
- removed JP3: PTSA-1.5/4-3.5FOST-TE-3.5-4P, synfinatic:PTSA-1.5/4-3.5FOST-TE-3.5-4P
- added C3: .01uf, Seeed-OPL-Capacitor:CERAMIC-1UF-25V-10%-X7R(0805)
- added C5, C6: 100uF, SparkFun-Capacitors:CAP_POLPTH1
- added Q1: IRLML6344, synfinatic:IRLML6344
- added R10: 1k, Seeed-OPL-Resistor:SMD-RES-10K-1%-1/8W(0805)
- added R3: 510, Seeed-OPL-Resistor:SMD-RES-10K-1%-1/8W(0805)
- added R8: 1k, Seeed-OPL-Resistor:SMD-RES-100K-1%-1/8W(0805)
- added U$4: TERM-BLOCK-P6-3.5, synfinatic:TERM-BLOCK-P6-3.5
Connections:
- new net GPIO_CTRL: Q1.G, R10.2
- new net SHDN: C5.+, C6.+, R3.1, U$2.SHDN
- new net V_BATT: U$2.VIN, U$4.P$5
- net +12V: now also R10.1, R3.2; no longer U$2.VIN
- net 3.3V: now also Q1.D
- net GND: now also C3.1, C5.-, C6.-, R8.1, U$4.P$1, U$4.P$6; no longer JP3.P$1
- net GPIO0: now also C3.2, Q1.S, R8.2
- net INPUT: now also U$4.P$3; no longer JP3.P$3
- net N$6: now also U$4.P$4; no longer JP3.P$4
- net OUTPUT: now also U$4.P$2; no longer JP3.P$2
Other:
- moved on the sheet: C2, D2, R4, R5, U$2, U$3
