File: GoProControl/goprocontrol.brd (EAGLE design)
At the start: 54.2 x 51.8 mm, 19 parts

Commit message: small board tweaks
Parts:
- removed JP3: PTSA-1.5/4-3.5FOST-TE-3.5-4P, synfinatic:TERM-4P-3.5
- added C3: .01uf, Seeed-OPL-Capacitor:C0805
- added C5, C6: 100uF, SparkFun-Capacitors:CPOL-RADIAL-100UF-25V
- added Q1: IRLML6344, synfinatic:SOT23
- added R10, R8: 1k, Seeed-OPL-Resistor:R0805
- added R3: 510, Seeed-OPL-Resistor:R0805
- added U$4: TERM-BLOCK-P6-3.5, synfinatic:TERM-6P-3.5
- moved U$2 13.0 mm to (19.0, 38.0)
- moved R5 10.8 mm to (37.5, 32.9)
- moved R2 9.06 mm to (16.8, 20.2)
- moved R1 9.00 mm to (20.4, 20.1)
- moved D2 8.54 mm to (40.0, 24.8)
- moved D3 7.88 mm to (50.7, 33.5), turned to 0 degrees
- moved C2 7.28 mm to (45.9, 13.8)
- moved D1 6.82 mm to (44.4, 33.2), turned to 90 degrees
- moved R4 5.39 mm to (39.9, 15.5)
- moved U$3 2.00 mm to (44.8, 23.1)
Connections:
- new net GPIO_CTRL: Q1.1, R10.2
- new net SHDN: C5.1, C6.1, R3.1, U$2.SHDN
- new net V_BATT: U$2.VIN, U$4.5
- net +12V: now also R10.1, R3.2; no longer U$2.VIN
- net 3.3V: now also Q1.3
- net GND: now also C3.1, C5.2, C6.2, R8.1, U$4.1, U$4.6; no longer JP3.1
- net GPIO0: now also C3.2, Q1.2, R8.2
- net INPUT: now also U$4.3; no longer JP3.3
- net N$6: now also U$4.4; no longer JP3.4
- net OUTPUT: now also U$4.2; no longer JP3.2
Routing:
- net 3.3V: track 55.5 -> 0.00 mm
- net 3.3V-TX: track 51.9 -> 0.00 mm
- net GPIO2: track 48.0 -> 0.00 mm, vias 1 -> 0
- net N$3: track 39.6 -> 0.00 mm
- net +12V: track 38.6 -> 0.00 mm
- net N$4: track 32.1 -> 0.00 mm
- net N$1: track 29.1 -> 0.00 mm
- net RXD: track 28.6 -> 0.00 mm
- net GPIO0: track 24.0 -> 0.00 mm
- net OUTPUT: track 23.9 -> 0.00 mm
- net TXD: track 14.8 -> 0.00 mm
- net GND: track 12.0 -> 0.00 mm, vias 1 -> 0
- net INPUT: track 9.34 -> 0.00 mm
- net 5V-TX: track 9.33 -> 0.00 mm
- net N$6: track 7.27 -> 0.00 mm
Other:
- board text added: "+"
- board text added: "12V"
- board text added: "SW12V"
- board text removed: "5-12V"
